File: cm300-board.kicad_sch (KiCad schematic)
At the start: 13 parts, among them J1 Screw_Terminal_01x02, J2 Screw_Terminal_01x02, J3 Conn_01x04_Female

Commit message: feat: convert to SMD, add Rge
Parts:
- D1, D3: footprint Diode_SMD:D_SOD-123F -> Diode_SMD:D_SOD-123; MPN (none) -> 1N5819HW-7-F
- D2, D4: footprint Diode_SMD:D_SMB -> Diode_SMD:D_SMC; MPN (none) -> SMCJ1.5KE24CA-TP
- J1, J2: footprint TerminalBlock_TE-Connectivity:TerminalBlock_TE_282834-2_1x02_P2.54mm_Horizontal -> Connector_Molex:Molex_KK-254_AE-6410-02A_1x02_P2.54mm_Vertical; MPN (none) -> 0022272021
- J3: MPN (none) -> 3534; digikey (none) -> 36-3534-ND
- R1, R4: MPN (none) -> CRM2512-FX-5R10ELF
- R2, R3: MPN (none) -> CRM2512-FX-R820ELF
- R5, R6: MPN (none) -> RMCF1206FT10K0
Other:
- title: (none) -> CM300DY-24H Gate Drive
Changed lines of the file:
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@@
 (kicad_sch (version 20230121) (generator eeschema)
   (paper "A4")
+  (title_block
+    (title "CM300DY-24H Gate Drive")
+    (date "2024-01-13")
+    (rev "v0.3.0")
+  )
   (junction (at 100.33 69.85) (diameter 0) (color 0 0 0 0)
   )
@@
       (effects (font (size 1.27 1.27)) hide)
     )
+    (property "MPN" "CRM2512-FX-5R10ELF" (at 72.39 59.69 90)
+      (effects (font (size 1.27 1.27)) hide)
+    )
     (pin "1")
     (pin "2")
@@
       (effects (font (size 1.27 1.27)) hide)
     )
+    (property "MPN" "CRM2512-FX-R820ELF" (at 72.39 67.31 90)
+      (effects (font (size 1.27 1.27)) hide)
+    )
     (pin "1")
     (pin "2")
@@
       (effects (font (size 1.27 1.27)))
     )
-    (property "Footprint" "Diode_SMD:D_SOD-123F" (at 83.82 71.755 0)
+    (property "Footprint" "Diode_SMD:D_SOD-123" (at 83.82 71.755 0)
       (effects (font (size 1.27 1.27)) hide)
     )
@@
       (effects (font (size 1.27 1.27)) hide)
     )
+    (property "MPN" "1N5819HW-7-F" (at 83.82 67.31 0)
+      (effects (font (size 1.27 1.27)) hide)
+    )
     (pin "1")
     (pin "2")
@@
       (effects (font (size 1.27 1.27)))
     )
-    (property "Footprint" "Diode_SMD:D_SMB" (at 96.52 72.39 0)
+    (property "Footprint" "Diode_SMD:D_SMC" (at 96.52 72.39 0)
       (effects (font (size 1.27 1.27)) hide)
     )
@@
       (effects (font (size 1.27 1.27)) hide)
     )
+    (property "MPN" "SMCJ1.5KE24CA-TP" (at 96.52 67.31 0)
+      (effects (font (size 1.27 1.27)) hide)
+    )
     (pin "1")
     (pin "2")
@@
       (effects (font (size 1.27 1.27)) hide)
     )
-    (property "Footprint" "TerminalBlock_TE-Connectivity:TerminalBlock_TE_282834-2_1x02_P2.54mm_Horizontal" (at 54.61 67.31 0)
+    (property "Footprint" "Connector_Molex:Molex_KK-254_AE-6410-02A_1x02_P2.54mm_Vertical" (at 54.61 67.31 0)
       (effects (font (size 1.27 1.27)) hide)
     )
@@
       (effects (font (size 1.27 1.27)) hide)
     )
+    (property "MPN" "0022272021" (at 54.61 67.31 0)
+      (effects (font (size 1.27 1.27)) hide)
+    )
     (pin "1")
     (pin "2")
@@
       (effects (font (size 1.27 1.27)) hide)
     )
+    (property "MPN" "CRM2512-FX-5R10ELF" (at 72.39 90.17 90)
+      (effects (font (size 1.27 1.27)) hide)
+    )
     (pin "1")
     (pin "2")
@@
       (effects (font (size 1.27 1.27)) hide)
     )
+    (property "MPN" "CRM2512-FX-R820ELF" (at 72.39 82.55 90)
+      (effects (font (size 1.27 1.27)) hide)
+    )
     (pin "1")
     (pin "2")
@@
       (effects (font (size 1.27 1.27)))
     )
-    (property "Footprint" "Diode_SMD:D_SOD-123F" (at 83.82 78.105 0)
+    (property "Footprint" "Diode_SMD:D_SOD-123" (at 83.82 78.105 0)
       (effects (font (size 1.27 1.27)) hide)
     )
@@
       (effects (font (size 1.27 1.27)) hide)
     )
+    (property "MPN" "1N5819HW-7-F" (at 83.82 82.55 0)
+      (effects (font (size 1.27 1.27)) hide)
+    )
     (pin "1")
     (pin "2")
@@
       (effects (font (size 1.27 1.27)))
     )
-    (property "Footprint" "Diode_SMD:D_SMB" (at 96.52 77.47 0)
+    (property "Footprint" "Diode_SMD:D_SMC" (at 96.52 77.47 0)
       (effects (font (size 1.27 1.27)) hide)
     )
@@
       (effects (font (size 1.27 1.27)) hide)
     )
+    (property "MPN" "SMCJ1.5KE24CA-TP" (at 96.52 82.55 0)
+      (effects (font (size 1.27 1.27)) hide)
+    )
+    (property "Field5" "" (at 96.52 82.55 0)
+      (effects (font (size 1.27 1.27)) hide)
+    )
     (pin "1")
     (pin "2")
@@
       (effects (font (size 1.27 1.27)) hide)
     )
-    (property "Footprint" "TerminalBlock_TE-Connectivity:TerminalBlock_TE_282834-2_1x02_P2.54mm_Horizontal" (at 54.61 80.01 0)
+    (property "Footprint" "Connector_Molex:Molex_KK-254_AE-6410-02A_1x02_P2.54mm_Vertical" (at 54.61 80.01 0)
       (effects (font (size 1.27 1.27)) hide)
     )
     (property "Datasheet" "~" (at 54.61 80.01 0)
+      (effects (font (size 1.27 1.27)) hide)
+    )
+    (property "MPN" "0022272021" (at 54.61 80.01 0)
       (effects (font (size 1.27 1.27)) hide)
     )
@@
       (effects (font (size 1.27 1.27)) hide)
     )
+    (property "MPN" "3534" (at 116.84 73.66 0)
+      (effects (font (size 1.27 1.27)) hide)
+    )
+    (property "digikey" "36-3534-ND" (at 116.84 73.66 0)
+      (effects (font (size 1.27 1.27)) hide)
+    )
     (pin "1")
     (pin "2")
@@
       (effects (font (size 1.27 1.27)) hide)
     )
+    (property "MPN" "RMCF1206FT10K0" (at 107.95 82.55 0)
+      (effects (font (size 1.27 1.27)) hide)
+    )
     (pin "1")
     (pin "2")
@@
       (effects (font (size 1.27 1.27)) hide)
     )
+    (property "MPN" "RMCF1206FT10K0" (at 107.95 67.31 0)
+      (effects (font (size 1.27 1.27)) hide)
+    )
